Commit message: feat: 导入魔法原子Z1的urdf文件并添加基础训练配置

File: legged_gym/resources/robots/Z1/MagicBotZ1_23dof.urdf (robot description, URDF)
Before this commit: robot MagicBotZ1, 31 links, 30 joints
Links:
- link left_ankle_roll_link: geometry collision box size=0.21622 0.050 0.02; visual mesh filename=meshes/left_ankle_roll_link.STL
- link right_ankle_roll_link: geometry collision box size=0.21622 0.050 0.02; visual mesh filename=meshes/right_ankle_roll_link.STL
